File: STM32F401RE lite board.kicad_pcb (KiCad board)
At the start: 2 copper layers, 62.8 x 41 mm, 40 parts, among them J2 USB_C_Receptacle_USB2.0_16P, J3 Conn_01x05_Pin, J6 Conn_01x24_Pin, J9 Conn_01x24_Pin, SW3 SW_SPST, SW4 SW_SPST, U2 LD3985M33R_SOT23, U3 STM32F401RETx, Y1 8MHz(16pF)

Commit message: C17
Parts:
- removed C12: 1nF, Capacitor_SMD:C_0402_1005Metric
- removed R4: 1MΩ, Resistor_SMD:R_0402_1005Metric
- added U1: USBLC6-2P6, Package_TO_SOT_SMD:SOT-666, F.Cu at (167.5, 87.5)
- moved R1 3.74 mm to (171.5, 80.9)
- moved R7 0.85 mm to (167.9, 84.3)
- moved D2 0.85 mm to (166.4, 84.7)
- moved R3 0.49 mm to (174.5, 80.9)
Connections:
- J2 pad A6: /D + -> /USB_D +
- J2 pad A7: /D - -> /USB_D -
- J2 pad B6: /D + -> /USB_D +
- J2 pad B7: /D - -> /USB_D -
- J2 pad S1: Net-(J2-SHIELD) -> GND
- R1 pad 1: Net-(J2-CC1) -> GND
- R1 pad 2: GND -> Net-(J2-CC2)
- R3 pad 1: GND -> Net-(J2-CC1)
- R3 pad 2: Net-(J2-CC2) -> GND
Routing:
- net Net-(J2-SHIELD): track 20.6 -> 0.00 mm
- net GND: track 90.4 -> 103.7 mm, vias 18 -> 17
- net /D +: track 12.7 -> 5.28 mm
- net /D -: track 11.8 -> 5.52 mm
- net /USB_D +: track 0.00 -> 5.98 mm
- net /USB_D -: track 0.00 -> 5.13 mm
- net VBUS: track 25.5 -> 29.2 mm
- net +3.3V: track 209.1 -> 211.7 mm
- net Net-(J2-CC2): track 7.31 -> 9.67 mm
- net /PWR_LED K: track 2.29 -> 1.63 mm
Other:
- board size 62.8 x 41 mm -> 62.6 x 41 mm
