File: STM32F401RE lite board.kicad_sch (KiCad schematic)
At the start: 39 parts, among them J2 USB_C_Receptacle_USB2.0_16P, J3 Conn_01x05_Pin, J6 Conn_01x24_Pin, J9 Conn_01x24_Pin, SW3 SW_SPST, SW4 SW_SPST, U2 LD3985M33R_SOT23, U3 STM32F401RETx, Y1 8MHz(16pF)

Commit message: C17
Parts:
- removed C12: 1nF, Capacitor_SMD:C_0402_1005Metric, symbol Device:C
- removed R4: 1MΩ, Resistor_SMD:R_0402_1005Metric, symbol Device:R
- added U1: USBLC6-2P6, Package_TO_SOT_SMD:SOT-666, symbol Power_Protection:USBLC6-2P6
Connections:
- net D +: now also U1.4 (I/O2); no longer J2.A6 (D+), J2.B6 (D+)
- net D -: now also U1.6 (I/O1); no longer J2.A7 (D-), J2.B7 (D-)
- net GND: now also J2.S1 (SHIELD), R1.1, R3.2, U1.2 (GND); no longer R1.2, R3.1
- net VBUS: now also U1.5 (VBUS)
- net at J2.A5 (CC1): now also R3.1; no longer R1.1
- net at J2.B5 (CC2): now also R1.2; no longer R3.2
- new net USB_D +: J2.A6 (D+), J2.B6 (D+), U1.3 (I/O2)
- new net USB_D -: J2.A7 (D-), J2.B7 (D-), U1.1 (I/O1)
Other:
- moved on the sheet: R1, R3
